File: stormkb47.kicad_sch (KiCad schematic)
At the start: 95 parts, among them J1 Conn_02x20_Odd_Even

Commit message: use proper-sized footprints for wide keys and add menu button
Parts:
- added D44: D_Small, Diode_SMD:D_SOD-123, symbol Device:D_Small
- added MX43: Menu, MX_Alps_Hybrid:MX-1U-NoLED, symbol MX_Alps_Hybrid:MX-NoLED
- MX1: value MX-NoLED -> Esc ~ `
- MX10: value MX-NoLED -> O ( 9
- MX11: value MX-NoLED -> P ) 0
- MX12: value MX-NoLED -> { [ _ -
- MX13: value MX-NoLED -> ] } + =
- MX14: value MX-NoLED -> Tab; footprint MX_Alps_Hybrid:MX-1U-NoLED -> MX_Alps_Hybrid:MX-1.5U-NoLED
- MX15: value MX-NoLED -> A F1
- MX16: value MX-NoLED -> S F2
- MX17: value MX-NoLED -> D F3
- MX18: value MX-NoLED -> F F4
- MX19: value MX-NoLED -> G F5
- MX2: value MX-NoLED -> Q ! 1
- MX20: value MX-NoLED -> H F6
- MX21: value MX-NoLED -> J F7
- MX22: value MX-NoLED -> K F8
- MX23: value MX-NoLED -> L F9
- MX24: value MX-NoLED -> ; : " '
- MX25: value MX-NoLED -> Enter; footprint MX_Alps_Hybrid:MX-1U-NoLED -> MX_Alps_Hybrid:MX-1.5U-NoLED
- MX26: value MX-NoLED -> Shift; footprint MX_Alps_Hybrid:MX-1U-NoLED -> MX_Alps_Hybrid:MX-2U-NoLED
- MX27: value MX-NoLED -> Z Ins
- MX28: value MX-NoLED -> X Del
- MX29: value MX-NoLED -> C Break
- MX3: value MX-NoLED -> W @ 2
- MX30: value MX-NoLED -> V Pause
- MX31: value MX-NoLED -> B PrtSc
- MX32: value MX-NoLED -> N SysRq
- MX33: value MX-NoLED -> M F10
- MX34: value MX-NoLED -> < , F11
- MX35: value MX-NoLED -> > . F12
- MX36: value MX-NoLED -> UpArr PgUp
- MX37: value MX-NoLED -> ? /
- MX38: value MX-NoLED -> Ctrl
- MX39: value MX-NoLED -> Fn
- MX4: value MX-NoLED -> E # 3
- MX40: value MX-NoLED -> Meta
- MX41: value MX-NoLED -> Alt
- MX42: value MX-NoLED -> Space; footprint MX_Alps_Hybrid:MX-1U-NoLED -> MX_Alps_Hybrid:MX-3U-NoLED
- MX44: renamed from MX43; value MX-NoLED -> AltGr
- MX45: renamed from MX44; value MX-NoLED -> | \
- MX46: renamed from MX45; value MX-NoLED -> ArrL Home
- MX47: renamed from MX46; value MX-NoLED -> ArrDn PgDn
- MX48: renamed from MX47; value MX-NoLED -> ArrR End
- MX5: value MX-NoLED -> R $ 4
- MX6: value MX-NoLED -> T % 5
- MX7: value MX-NoLED -> Y ^ 6
- MX8: value MX-NoLED -> U & 7
- MX9: value MX-NoLED -> I * 8
- renumbered D44 to D45, D45 to D46, D46 to D47, D47 to D48
Connections:
- net COL6: now also MX42.1 (COL)
- net COL7: no longer MX42.1 (COL)
- net COL8: now also MX43.1 (COL)
- net ROW4: now also D44.1 (K)
- net at D43.2 (A): now also MX43.2 (ROW); no longer MX44.2 (ROW)
- new net: D44.2 (A), MX44.2 (ROW)
Other:
- note added: "Menu"
- moved on the sheet: D42, D43, MX42
